File: eagle/vceg.brd (EAGLE design)
At the start: 100 x 80 mm, 71 parts, among them IC1 4052N, IC2 4001N, IC3 TL074P, IC4 LM13700N, Q1 2N3906INLINE, Q2 2N3906INLINE, T1 2N3904, U1 POWER

Commit message: improved layout
Parts:
- moved LED1 19.0 mm to (93.2, 64.3), turned to 90 degrees
- moved R22 8.81 mm to (12.2, 28.2)
- moved TG_SWA_1 6.23 mm to (88.9, 44.7)
- moved ATTACK 5.95 mm to (9.14, 15.7)
- moved R7 2.84 mm to (80.3, 62.5)
- moved LEVEL 2.34 mm to (81.0, 66.0)
- moved R10 2.27 mm to (91.7, 54.1), turned to 270 degrees
- moved TG_SWA_3 2.16 mm to (67.6, 69.3)
- moved C8 1.98 mm to (17.8, 23.9)
- moved GATE_NORMAL 1.61 mm to (18.8, 52.6)
- moved R18 1.37 mm to (29.0, 47.0)
- moved R1 1.27 mm to (12.4, 41.9)
- moved TG_SWB_1 1.02 mm to (28.2, 42.7)
- moved U1 1.02 mm to (11.2, 64.0)
- moved IC4 1.02 mm to (45.5, 65.3)
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Routing:
- net GND: track 612.4 -> 571.9 mm
- net +12V: track 470.9 -> 437.3 mm
- net N$5: track 138.0 -> 126.7 mm
- net N$44: track 14.9 -> 6.13 mm
- net N$40: track 21.7 -> 18.5 mm
- net N$22: track 18.4 -> 21.3 mm
- net N$43: track 17.0 -> 14.5 mm
- net N$26: track 67.1 -> 64.8 mm
- net -12V: track 124.2 -> 126.1 mm
- net N$10: track 2.96 -> 4.71 mm
- net N$23: track 7.59 -> 9.26 mm
- net N$28: track 36.3 -> 37.7 mm
- net N$16: track 21.5 -> 20.2 mm
- net N$21: track 5.76 -> 4.49 mm
- net N$33: track 10.2 -> 11.4 mm
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